Commit message: new features, code tided, added weight, classes, optuna

File: models/ur10/ur10_sandbox.urdf (robot description, URDF)
Before this commit: robot ur10, 14 links, 13 joints
Links:
- removed link box_link
- added link ee_link, mass 0.001; collision box size=0.01 0.01 0.01
- added link left_inner_finger, mass 0.00724255; collision mesh filename=collision/robotiq_85_gripper/inner_finger_coarse.STL
- added link left_inner_knuckle, mass 0.0110931; collision mesh filename=collision/robotiq_85_gripper/inner_knuckle_coarse.STL
- added link right_inner_finger, mass 0.00724255; collision mesh filename=collision/robotiq_85_gripper/inner_finger_coarse.STL
- added link right_inner_knuckle, mass 0.0110931; collision mesh filename=collision/robotiq_85_gripper/inner_knuckle_coarse.STL
- added link robotiq_85_base_link, mass 0.30915; collision mesh filename=collision/robotiq_85_gripper/robotiq_85_base_link_coarse.STL
Joints:
- removed joint tool0_to_box
- added joint base_to_lik: type revolute, parent robotiq_85_base_link, child left_inner_knuckle, origin xyz=0.0127 0 0.0693075 rpy=0 0 0, axis 0 1 0, limit lower=-1 upper=1 effort=1000 velocity=10
- added joint base_to_rik: type revolute, parent robotiq_85_base_link, child right_inner_knuckle, origin xyz=-0.0127 0 0.0693075 rpy=0 0 3.14159, axis 0 1 0, limit lower=-1 upper=1 effort=1000 velocity=10
- added joint ee_link-robotiq_85_base_link: type fixed, parent ee_link, child robotiq_85_base_link, origin xyz=0 0 0 rpy=1.5708 0 1.5708
- added joint left_knuckle-left_finger: type fixed, parent left_inner_knuckle, child left_inner_finger, origin xyz=0.0345853 0 0.045497 rpy=0 0 0
- added joint right_knuckle-right_finger: type fixed, parent right_inner_knuckle, child right_inner_finger, origin xyz=0.034106 0 0.0458574 rpy=0 0 0
- added joint wrist_3_link-ee_link: type fixed, parent wrist_3_link, child ee_link, origin xyz=0 0 0 rpy=0 -1.5708 3.14159
